File: di_simplified/di_simplified.sch (KiCad schematic (older format))
At the start: 16 parts

Commit message: layout stuff
Connections:
- net GND: now also U?.7; no longer C?.1, R?.1, R?.2, U?.5 (+)
- new net: C?.1, R?.1, R?.2, U?.5 (+)
- no-connect marks 2 -> 1
Other:
- note added: "Split-rail reference and buffer"
- note removed: "Bias reference"
- moved on the sheet: C?, R?, U?B
Changed lines of the file:
@@
 L R R?
 U 1 1 5744D148
-P 3200 1750
-F 0 "R?" H 3270 1796 50  0000 L CNN
-F 1 "100k" H 3270 1704 50  0000 L CNN
-F 2 "" V 3130 1750 50  0000 C CNN
-F 3 "" H 3200 1750 50  0000 C CNN
-	1    3200 1750
+P 3300 1500
+F 0 "R?" H 3370 1546 50  0000 L CNN
+F 1 "100k" H 3370 1454 50  0000 L CNN
+F 2 "" V 3230 1500 50  0000 C CNN
+F 3 "" H 3300 1500 50  0000 C CNN
+	1    3300 1500
 	1    0    0    -1
 $EndComp
@@
 L R R?
 U 1 1 5744D1B2
-P 3200 2150
-F 0 "R?" H 3270 2196 50  0000 L CNN
-F 1 "100k" H 3270 2104 50  0000 L CNN
-F 2 "" V 3130 2150 50  0000 C CNN
-F 3 "" H 3200 2150 50  0000 C CNN
-	1    3200 2150
+P 3300 1900
+F 0 "R?" H 3370 1946 50  0000 L CNN
+F 1 "100k" H 3370 1854 50  0000 L CNN
+F 2 "" V 3230 1900 50  0000 C CNN
+F 3 "" H 3300 1900 50  0000 C CNN
+	1    3300 1900
 	1    0    0    -1
 $EndComp
@@
 Text Notes 4950 3850 0    60   ~ 0
 Preamp buffer
-Text Notes 3150 2700 0    60   ~ 0
-Bias reference
-Wire Wire Line
-	3200 1900 3200 2000
-Wire Wire Line
-	3200 1950 4050 1950
-Connection ~ 3200 1950
+Text Notes 3450 2450 0    60   ~ 0
+Split-rail reference and buffer
+Wire Wire Line
+	3300 1650 3300 1750
+Wire Wire Line
+	3300 1700 4150 1700
+Connection ~ 3300 1700
 Wire Wire Line
 	4950 3200 5150 3200
@@
 L C C?
 U 1 1 57450564
-P 3550 2150
-F 0 "C?" H 3665 2196 50  0000 L CNN
-F 1 "100n" H 3665 2104 50  0000 L CNN
-F 2 "" H 3588 2000 50  0000 C CNN
-F 3 "" H 3550 2150 50  0000 C CNN
-	1    3550 2150
-	1    0    0    -1
-$EndComp
-Wire Wire Line
-	3550 1950 3550 2000
-Connection ~ 3550 1950
+P 3650 1900
+F 0 "C?" H 3765 1946 50  0000 L CNN
+F 1 "100n" H 3765 1854 50  0000 L CNN
+F 2 "" H 3688 1750 50  0000 C CNN
+F 3 "" H 3650 1900 50  0000 C CNN
+	1    3650 1900
+	1    0    0    -1
+$EndComp
+Wire Wire Line
+	3650 1700 3650 1750
+Connection ~ 3650 1700
 $Comp
 L NE5532 U?
 U 2 1 5746D07A
-P 5450 2000
-F 0 "U?" H 5791 2046 50  0000 L CNN
-F 1 "LM358N" H 5791 1954 50  0000 L CNN
-F 2 "" H 5450 2000 50  0000 C CNN
-F 3 "" H 5450 2000 50  0000 C CNN
-	2    5450 2000
+P 4450 1800
+F 0 "U?" H 4791 1846 50  0000 L CNN
+F 1 "LM358N" H 4791 1754 50  0000 L CNN
+F 2 "" H 4450 1800 50  0000 C CNN
+F 3 "" H 4450 1800 50  0000 C CNN
+	2    4450 1800
 	1    0    0    -1
 $EndComp
@@
 L GND #PWR?
 U 1 1 5746D137
-P 5050 2200
-F 0 "#PWR?" H 5050 1950 50  0001 C CNN
-F 1 "GND" H 5058 2026 50  0000 C CNN
-F 2 "" H 5050 2200 50  0000 C CNN
-F 3 "" H 5050 2200 50  0000 C CNN
-	1    5050 2200
-	1    0    0    -1
-$EndComp
-Wire Wire Line
-	5050 1900 5050 2200
-Wire Wire Line
-	5050 2100 5150 2100
-Wire Wire Line
-	5050 1900 5150 1900
-Connection ~ 5050 2100
+P 5200 1800
+F 0 "#PWR?" H 5200 1550 50  0001 C CNN
+F 1 "GND" H 5208 1626 50  0000 C CNN
+F 2 "" H 5200 1800 50  0000 C CNN
+F 3 "" H 5200 1800 50  0000 C CNN
+	1    5200 1800
+	1    0    0    -1
+$EndComp
 $Comp
 L GND #PWR?
@@
 $EndComp
 $Comp
-L GND #PWR?
-U 1 1 5748440B
-P 4050 2000
-F 0 "#PWR?" H 4050 1750 50  0001 C CNN
-F 1 "GND" H 4058 1826 50  0000 C CNN
-F 2 "" H 4050 2000 50  0000 C CNN
-F 3 "" H 4050 2000 50  0000 C CNN
-	1    4050 2000
-	1    0    0    -1
-$EndComp
-Wire Wire Line
-	4050 1950 4050 2000
-$Comp
 L VSS #PWR?
 U 1 1 57484564
-P 3200 2300
-F 0 "#PWR?" H 3200 2150 50  0001 C CNN
-F 1 "VSS" H 3221 2474 50  0000 C CNN
-F 2 "" H 3200 2300 50  0000 C CNN
-F 3 "" H 3200 2300 50  0000 C CNN
-	1    3200 2300
+P 3300 2050
+F 0 "#PWR?" H 3300 1900 50  0001 C CNN
+F 1 "VSS" H 3321 2224 50  0000 C CNN
+F 2 "" H 3300 2050 50  0000 C CNN
+F 3 "" H 3300 2050 50  0000 C CNN
+	1    3300 2050
 	-1   0    0    1
 $EndComp
@@
 L VDD #PWR?
 U 1 1 57484615
-P 3200 1600
-F 0 "#PWR?" H 3200 1450 50  0001 C CNN
-F 1 "VDD" H 3220 1774 50  0000 C CNN
-F 2 "" H 3200 1600 50  0000 C CNN
-F 3 "" H 3200 1600 50  0000 C CNN
-	1    3200 1600
+P 3300 1350
+F 0 "#PWR?" H 3300 1200 50  0001 C CNN
+F 1 "VDD" H 3320 1524 50  0000 C CNN
+F 2 "" H 3300 1350 50  0000 C CNN
+F 3 "" H 3300 1350 50  0000 C CNN
+	1    3300 1350
 	1    0    0    -1
 $EndComp
@@
 L VSS #PWR?
 U 1 1 57484650
-P 3550 2300
-F 0 "#PWR?" H 3550 2150 50  0001 C CNN
-F 1 "VSS" H 3571 2474 50  0000 C CNN
-F 2 "" H 3550 2300 50  0000 C CNN
-F 3 "" H 3550 2300 50  0000 C CNN
-	1    3550 2300
+P 3650 2050
+F 0 "#PWR?" H 3650 1900 50  0001 C CNN
+F 1 "VSS" H 3671 2224 50  0000 C CNN
+F 2 "" H 3650 2050 50  0000 C CNN
+F 3 "" H 3650 2050 50  0000 C CNN
+	1    3650 2050
 	-1   0    0    1
 $EndComp
@@
 L VSS #PWR?
 U 1 1 57484F59
-P 5350 2300
-F 0 "#PWR?" H 5350 2150 50  0001 C CNN
-F 1 "VSS" H 5371 2474 50  0000 C CNN
-F 2 "" H 5350 2300 50  0000 C CNN
-F 3 "" H 5350 2300 50  0000 C CNN
-	1    5350 2300
+P 4350 2100
+F 0 "#PWR?" H 4350 1950 50  0001 C CNN
+F 1 "VSS" H 4371 2274 50  0000 C CNN
+F 2 "" H 4350 2100 50  0000 C CNN
+F 3 "" H 4350 2100 50  0000 C CNN
+	1    4350 2100
 	-1   0    0    1
 $EndComp
@@
 L VDD #PWR?
 U 1 1 57484FC8
-P 5350 1700
-F 0 "#PWR?" H 5350 1550 50  0001 C CNN
-F 1 "VDD" H 5370 1874 50  0000 C CNN
-F 2 "" H 5350 1700 50  0000 C CNN
-F 3 "" H 5350 1700 50  0000 C CNN
-	1    5350 1700
+P 4350 1500
+F 0 "#PWR?" H 4350 1350 50  0001 C CNN
+F 1 "VDD" H 4370 1674 50  0000 C CNN
+F 2 "" H 4350 1500 50  0000 C CNN
+F 3 "" H 4350 1500 50  0000 C CNN
+	1    4350 1500
 	1    0    0    -1
 $EndComp
@@
 	-1   0    0    1
 $EndComp
-NoConn ~ 5750 2000
 $Comp
 L NE5532 U?
@@
 Connection ~ 8150 2350
 Connection ~ 8150 3650
+Wire Wire Line
+	4150 1900 4150 2350
+Wire Wire Line
+	4150 2350 4750 2350
+Wire Wire Line
+	4750 2350 4750 1800
+Wire Wire Line
+	4750 1800 5200 1800
+Connection ~ 4750 1800
 $EndSCHEMATC
