File: breadbox/breadbox.kicad_pcb (KiCad board)
At the start: 2 copper layers, 50 x 50 mm, 48 parts, among them P1 IN, P10 3+, P11 3-, P12 1OUT, P13 2OUT, P14 3OUT, P15 CONN, P16 CONN, P17 CONN, P18 CONN, P19 CONN, P2 OUT, P20 CONN, P21 VDD, P22 CONN, P23 GND, P24 CONN, P25 VSS, P26 4+, P27 4-, P28 5-, P29 5+, P3 PP3, P30 4OUT, P31 5OUT, P4 IN, P5 OUT, P6 1+, P7 1-, P8 2+, P9 2-, U1 LM358N, U2 LM358N, U3 LM358N, U4 LM358N

Commit message: Added C5, changed M3-mount to M3 hole
Parts:
- removed the REF** at (55.0, 55.0)
- removed the REF** at (95.0, 55.0)
- removed the REF** at (95.0, 95.0)
- removed the REF** at (55.0, 95.0)
- added REF**: M3_HOLE, agg:M3_HOLE, F.Cu at (55.0, 95.0)
- added REF**: M3_HOLE, agg:M3_HOLE, F.Cu at (55.0, 55.0)
- added REF**: M3_HOLE, agg:M3_HOLE, F.Cu at (95.0, 55.0)
- added REF**: M3_HOLE, agg:M3_HOLE, F.Cu at (95.0, 95.0)
Changed lines of the file:
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@@
   )
   (setup
-    (last_trace_width 0.4)
+    (last_trace_width 0.25)
     (user_trace_width 0.4)
     (user_trace_width 1)
@@
     (add_net VSS)
   )
+  (module agg:M3_HOLE (layer F.Cu)
+    (at 55 95)
+    (fp_text reference REF** (at 0 -2.5) (layer F.Fab) hide
+      (effects (font (size 1 1) (thickness 0.15)))
+    )
+    (fp_text value M3_HOLE (at 0 2.5) (layer F.Fab) hide
+      (effects (font (size 1 1) (thickness 0.15)))
+    )
+    (fp_line (start -1.8 1.8) (end -1.8 -1.8) (layer F.CrtYd) (width 0.01))
+    (fp_line (start 1.8 1.8) (end -1.8 1.8) (layer F.CrtYd) (width 0.01))
+    (fp_line (start 1.8 -1.8) (end 1.8 1.8) (layer F.CrtYd) (width 0.01))
+    (fp_line (start -1.8 -1.8) (end 1.8 -1.8) (layer F.CrtYd) (width 0.01))
+    (pad "" np_thru_hole circle (at 0 0) (size 3.2 3.2) (drill 3.2) (layers *.Cu F.Mask))
+  )
   (module Resistors_SMD:R_0603 (layer F.Cu)
     (at 69.596 54.61)
@@
       (rotate (xyz 0 0 0))
     )
-  )
-  (module agg:M3_MOUNT (layer F.Cu)
-    (at 55 55)
-    (fp_text reference REF** (at 0 -4.1) (layer F.Fab) hide
-      (effects (font (size 1 1) (thickness 0.15)))
-    )
-    (fp_text value M3_MOUNT (at 0 4.1) (layer F.Fab) hide
-      (effects (font (size 1 1) (thickness 0.15)))
-    )
-    (fp_line (start -3.4 3.4) (end -3.4 -3.4) (layer F.CrtYd) (width 0.01))
-    (fp_line (start 3.4 3.4) (end -3.4 3.4) (layer F.CrtYd) (width 0.01))
-    (fp_line (start 3.4 -3.4) (end 3.4 3.4) (layer F.CrtYd) (width 0.01))
-    (fp_line (start -3.4 -3.4) (end 3.4 -3.4) (layer F.CrtYd) (width 0.01))
-    (pad "" np_thru_hole circle (at 0 0) (size 3.3 3.3) (drill 3.3) (layers *.Cu *.Mask F.SilkS)
-      (solder_mask_margin 1.5) (clearance 1.65))
-    (pad "" np_thru_hole circle (at 0 -2.5) (size 0.6 0.6) (drill 0.6) (layers *.Cu *.Mask F.SilkS))
-    (pad "" np_thru_hole circle (at 2.5 0) (size 0.6 0.6) (drill 0.6) (layers *.Cu *.Mask F.SilkS))
-    (pad "" np_thru_hole circle (at 0 2.5) (size 0.6 0.6) (drill 0.6) (layers *.Cu *.Mask F.SilkS))
-    (pad "" np_thru_hole circle (at -2.5 0) (size 0.6 0.6) (drill 0.6) (layers *.Cu *.Mask F.SilkS))
-    (pad "" np_thru_hole circle (at -1.8 -1.8) (size 0.6 0.6) (drill 0.6) (layers *.Cu *.Mask F.SilkS))
-    (pad "" np_thru_hole circle (at 1.8 -1.8) (size 0.6 0.6) (drill 0.6) (layers *.Cu *.Mask F.SilkS))
-    (pad "" np_thru_hole circle (at -1.8 1.8) (size 0.6 0.6) (drill 0.6) (layers *.Cu *.Mask F.SilkS))
-    (pad "" np_thru_hole circle (at 1.8 1.8) (size 0.6 0.6) (drill 0.6) (layers *.Cu *.Mask F.SilkS))
-  )
-  (module agg:M3_MOUNT (layer F.Cu)
-    (at 95 55)
-    (fp_text reference REF** (at 0 -4.1) (layer F.Fab) hide
-      (effects (font (size 1 1) (thickness 0.15)))
-    )
-    (fp_text value M3_MOUNT (at 0 4.1) (layer F.Fab) hide
-      (effects (font (size 1 1) (thickness 0.15)))
-    )
-    (fp_line (start -3.4 3.4) (end -3.4 -3.4) (layer F.CrtYd) (width 0.01))
-    (fp_line (start 3.4 3.4) (end -3.4 3.4) (layer F.CrtYd) (width 0.01))
-    (fp_line (start 3.4 -3.4) (end 3.4 3.4) (layer F.CrtYd) (width 0.01))
-    (fp_line (start -3.4 -3.4) (end 3.4 -3.4) (layer F.CrtYd) (width 0.01))
-    (pad "" np_thru_hole circle (at 0 0) (size 3.3 3.3) (drill 3.3) (layers *.Cu *.Mask F.SilkS)
-      (solder_mask_margin 1.5) (clearance 1.65))
-    (pad "" np_thru_hole circle (at 0 -2.5) (size 0.6 0.6) (drill 0.6) (layers *.Cu *.Mask F.SilkS))
-    (pad "" np_thru_hole circle (at 2.5 0) (size 0.6 0.6) (drill 0.6) (layers *.Cu *.Mask F.SilkS))
-    (pad "" np_thru_hole circle (at 0 2.5) (size 0.6 0.6) (drill 0.6) (layers *.Cu *.Mask F.SilkS))
-    (pad "" np_thru_hole circle (at -2.5 0) (size 0.6 0.6) (drill 0.6) (layers *.Cu *.Mask F.SilkS))
-    (pad "" np_thru_hole circle (at -1.8 -1.8) (size 0.6 0.6) (drill 0.6) (layers *.Cu *.Mask F.SilkS))
-    (pad "" np_thru_hole circle (at 1.8 -1.8) (size 0.6 0.6) (drill 0.6) (layers *.Cu *.Mask F.SilkS))
-    (pad "" np_thru_hole circle (at -1.8 1.8) (size 0.6 0.6) (drill 0.6) (layers *.Cu *.Mask F.SilkS))
-    (pad "" np_thru_hole circle (at 1.8 1.8) (size 0.6 0.6) (drill 0.6) (layers *.Cu *.Mask F.SilkS))
-  )
-  (module agg:M3_MOUNT (layer F.Cu)
-    (at 95 95)
-    (fp_text reference REF** (at 0 -4.1) (layer F.Fab) hide
-      (effects (font (size 1 1) (thickness 0.15)))
-    )
-    (fp_text value M3_MOUNT (at 0 4.1) (layer F.Fab) hide
-      (effects (font (size 1 1) (thickness 0.15)))
-    )
-    (fp_line (start -3.4 3.4) (end -3.4 -3.4) (layer F.CrtYd) (width 0.01))
-    (fp_line (start 3.4 3.4) (end -3.4 3.4) (layer F.CrtYd) (width 0.01))
-    (fp_line (start 3.4 -3.4) (end 3.4 3.4) (layer F.CrtYd) (width 0.01))
-    (fp_line (start -3.4 -3.4) (end 3.4 -3.4) (layer F.CrtYd) (width 0.01))
-    (pad "" np_thru_hole circle (at 0 0) (size 3.3 3.3) (drill 3.3) (layers *.Cu *.Mask F.SilkS)
-      (solder_mask_margin 1.5) (clearance 1.65))
-    (pad "" np_thru_hole circle (at 0 -2.5) (size 0.6 0.6) (drill 0.6) (layers *.Cu *.Mask F.SilkS))
-    (pad "" np_thru_hole circle (at 2.5 0) (size 0.6 0.6) (drill 0.6) (layers *.Cu *.Mask F.SilkS))
-    (pad "" np_thru_hole circle (at 0 2.5) (size 0.6 0.6) (drill 0.6) (layers *.Cu *.Mask F.SilkS))
-    (pad "" np_thru_hole circle (at -2.5 0) (size 0.6 0.6) (drill 0.6) (layers *.Cu *.Mask F.SilkS))
-    (pad "" np_thru_hole circle (at -1.8 -1.8) (size 0.6 0.6) (drill 0.6) (layers *.Cu *.Mask F.SilkS))
-    (pad "" np_thru_hole circle (at 1.8 -1.8) (size 0.6 0.6) (drill 0.6) (layers *.Cu *.Mask F.SilkS))
-    (pad "" np_thru_hole circle (at -1.8 1.8) (size 0.6 0.6) (drill 0.6) (layers *.Cu *.Mask F.SilkS))
-    (pad "" np_thru_hole circle (at 1.8 1.8) (size 0.6 0.6) (drill 0.6) (layers *.Cu *.Mask F.SilkS))
-  )
-  (module agg:M3_MOUNT (layer F.Cu)
-    (at 55 95)
-    (fp_text reference REF** (at 0 -4.1) (layer F.Fab) hide
-      (effects (font (size 1 1) (thickness 0.15)))
-    )
-    (fp_text value M3_MOUNT (at 0 4.1) (layer F.Fab) hide
-      (effects (font (size 1 1) (thickness 0.15)))
-    )
-    (fp_line (start -3.4 3.4) (end -3.4 -3.4) (layer F.CrtYd) (width 0.01))
-    (fp_line (start 3.4 3.4) (end -3.4 3.4) (layer F.CrtYd) (width 0.01))
-    (fp_line (start 3.4 -3.4) (end 3.4 3.4) (layer F.CrtYd) (width 0.01))
-    (fp_line (start -3.4 -3.4) (end 3.4 -3.4) (layer F.CrtYd) (width 0.01))
-    (pad "" np_thru_hole circle (at 0 0) (size 3.3 3.3) (drill 3.3) (layers *.Cu *.Mask F.SilkS)
-      (solder_mask_margin 1.5) (clearance 1.65))
-    (pad "" np_thru_hole circle (at 0 -2.5) (size 0.6 0.6) (drill 0.6) (layers *.Cu *.Mask F.SilkS))
-    (pad "" np_thru_hole circle (at 2.5 0) (size 0.6 0.6) (drill 0.6) (layers *.Cu *.Mask F.SilkS))
-    (pad "" np_thru_hole circle (at 0 2.5) (size 0.6 0.6) (drill 0.6) (layers *.Cu *.Mask F.SilkS))
-    (pad "" np_thru_hole circle (at -2.5 0) (size 0.6 0.6) (drill 0.6) (layers *.Cu *.Mask F.SilkS))
-    (pad "" np_thru_hole circle (at -1.8 -1.8) (size 0.6 0.6) (drill 0.6) (layers *.Cu *.Mask F.SilkS))
-    (pad "" np_thru_hole circle (at 1.8 -1.8) (size 0.6 0.6) (drill 0.6) (layers *.Cu *.Mask F.SilkS))
-    (pad "" np_thru_hole circle (at -1.8 1.8) (size 0.6 0.6) (drill 0.6) (layers *.Cu *.Mask F.SilkS))
-    (pad "" np_thru_hole circle (at 1.8 1.8) (size 0.6 0.6) (drill 0.6) (layers *.Cu *.Mask F.SilkS))
   )
   (module breadbox:Pin_Header_Straight_1x03 (layer F.Cu)
@@
     (tags "capacitor 0603")
     (attr smd)
-    (fp_text reference C5 (at 0 -1.9) (layer F.SilkS)
+    (fp_text reference C5 (at 0 -1.9) (layer F.SilkS) hide
       (effects (font (size 1 1) (thickness 0.15)))
     )
@@
     )
   )
+  (module agg:M3_HOLE (layer F.Cu)
+    (at 55 55)
+    (fp_text reference REF** (at 0 -2.5) (layer F.Fab) hide
+      (effects (font (size 1 1) (thickness 0.15)))
+    )
+    (fp_text value M3_HOLE (at 0 2.5) (layer F.Fab) hide
+      (effects (font (size 1 1) (thickness 0.15)))
+    )
+    (fp_line (start -1.8 1.8) (end -1.8 -1.8) (layer F.CrtYd) (width 0.01))
+    (fp_line (start 1.8 1.8) (end -1.8 1.8) (layer F.CrtYd) (width 0.01))
+    (fp_line (start 1.8 -1.8) (end 1.8 1.8) (layer F.CrtYd) (width 0.01))
+    (fp_line (start -1.8 -1.8) (end 1.8 -1.8) (layer F.CrtYd) (width 0.01))
+    (pad "" np_thru_hole circle (at 0 0) (size 3.2 3.2) (drill 3.2) (layers *.Cu F.Mask))
+  )
+  (module agg:M3_HOLE (layer F.Cu)
+    (at 95 55)
+    (fp_text reference REF** (at 0 -2.5) (layer F.Fab) hide
+      (effects (font (size 1 1) (thickness 0.15)))
+    )
+    (fp_text value M3_HOLE (at 0 2.5) (layer F.Fab) hide
+      (effects (font (size 1 1) (thickness 0.15)))
+    )
+    (fp_line (start -1.8 1.8) (end -1.8 -1.8) (layer F.CrtYd) (width 0.01))
+    (fp_line (start 1.8 1.8) (end -1.8 1.8) (layer F.CrtYd) (width 0.01))
+    (fp_line (start 1.8 -1.8) (end 1.8 1.8) (layer F.CrtYd) (width 0.01))
+    (fp_line (start -1.8 -1.8) (end 1.8 -1.8) (layer F.CrtYd) (width 0.01))
+    (pad "" np_thru_hole circle (at 0 0) (size 3.2 3.2) (drill 3.2) (layers *.Cu F.Mask))
+  )
+  (module agg:M3_HOLE (layer F.Cu)
+    (at 95 95)
+    (fp_text reference REF** (at 0 -2.5) (layer F.Fab) hide
+      (effects (font (size 1 1) (thickness 0.15)))
+    )
+    (fp_text value M3_HOLE (at 0 2.5) (layer F.Fab) hide
+      (effects (font (size 1 1) (thickness 0.15)))
+    )
+    (fp_line (start -1.8 1.8) (end -1.8 -1.8) (layer F.CrtYd) (width 0.01))
+    (fp_line (start 1.8 1.8) (end -1.8 1.8) (layer F.CrtYd) (width 0.01))
+    (fp_line (start 1.8 -1.8) (end 1.8 1.8) (layer F.CrtYd) (width 0.01))
+    (fp_line (start -1.8 -1.8) (end 1.8 -1.8) (layer F.CrtYd) (width 0.01))
+    (pad "" np_thru_hole circle (at 0 0) (size 3.2 3.2) (drill 3.2) (layers *.Cu F.Mask))
+  )
   (gr_text BREADBOX (at 80.772 93.98) (layer B.SilkS)

Commit message: Breadbox schematic and finished PCB
Parts:
- P1, P5: footprint Pin_Headers:Pin_Header_Straight_1x02 -> Pin_Headers:Pin_Header_Straight_1x03
- moved P5 0.76 mm to (64.8, 97.5)
Routing:
- net Net-(P5-Pad2): track 9.64 -> 13.4 mm, vias 1 -> 0
- net Net-(P1-Pad2): track 4.28 -> 6.82 mm
- net VDD: track 167.5 -> 168.1 mm

Commit message: Final tweaks
Parts:
- added C6: 100n, agg:0603, F.Cu at (58.4, 78.7)
- added D1: LED, Pin_Headers:Pin_Header_Straight_1x02, F.Cu at (60.2, 52.1)
- added R5: R, agg:0603, F.Cu at (60.2, 58.2)
- moved P3 4.10 mm to (64.8, 52.1), turned to 0 degrees
Routing:
- net GND: track 32.8 -> 37.7 mm
- net Net-(D1-Pad2): track 0.00 -> 3.89 mm
- net VDD: track 168.1 -> 171.7 mm
- net VSS: track 177.9 -> 180.0 mm, vias 0 -> 1
Other:
- board text added: "LED"
