File: breadbox/breadbox.sch (KiCad schematic (older format))
At the start: 44 parts, among them P1 IN, P10 3+, P11 3-, P12 1OUT, P13 2OUT, P14 3OUT, P15 CONN, P16 CONN, P17 CONN, P18 CONN, P19 CONN, P2 OUT, P20 CONN, P21 VDD, P22 CONN, P23 GND, P24 CONN, P25 VSS, P26 4+, P27 4-, P28 5-, P29 5+, P3 PP3, P30 4OUT, P31 5OUT, P4 IN, P5 OUT, P6 1+, P7 1-, P8 2+, P9 2-, U1 LM358N, U2 LM358N, U3 LM358N, U4 LM358N

Commit message: Breadbox schematic and finished PCB
Parts:
- removed P1: IN, Pin_Headers:Pin_Header_Straight_1x02, symbol CONN_01X02
- removed P5: OUT, Pin_Headers:Pin_Header_Straight_1x02, symbol CONN_01X02
- added P1: IN, Pin_Headers:Pin_Header_Straight_1x03, symbol CONN_01X03
- added P5: OUT, Pin_Headers:Pin_Header_Straight_1x03, symbol CONN_01X03
Connections:
- net GND: now also P1.1 (P1), P5.1 (P1)
- net at R1.1: now also P1.2 (P2), P1.3 (P3)
- net at U1.1, U1.2 (-): now also P5.2 (P2), P5.3 (P3)
Changed lines of the file:
@@
 $EndComp
 $Comp
-L VSS #PWR01
+L VSS #PWR3
 U 1 1 574B33DE
 P 2000 1800
-F 0 "#PWR01" H 2000 1650 50  0001 C CNN
+F 0 "#PWR3" H 2000 1650 50  0001 C CNN
 F 1 "VSS" H 2021 1974 50  0000 C CNN
 F 2 "" H 2000 1800 50  0000 C CNN
@@
 $EndComp
 $Comp
-L VDD #PWR02
+L VDD #PWR2
 U 1 1 574B3403
 P 2000 1700
-F 0 "#PWR02" H 2000 1550 50  0001 C CNN
+F 0 "#PWR2" H 2000 1550 50  0001 C CNN
 F 1 "VDD" H 2020 1874 50  0000 C CNN
 F 2 "" H 2000 1700 50  0000 C CNN
@@
 $EndComp
 $Comp
-L VDD #PWR03
+L VDD #PWR7
 U 1 1 574B348D
 P 2500 1400
-F 0 "#PWR03" H 2500 1250 50  0001 C CNN
+F 0 "#PWR7" H 2500 1250 50  0001 C CNN
 F 1 "VDD" H 2520 1574 50  0000 C CNN
 F 2 "" H 2500 1400 50  0000 C CNN
@@
 $EndComp
 $Comp
-L VSS #PWR04
+L VSS #PWR8
 U 1 1 574B34AA
 P 2500 2100
-F 0 "#PWR04" H 2500 1950 50  0001 C CNN
+F 0 "#PWR8" H 2500 1950 50  0001 C CNN
 F 1 "VSS" H 2521 2274 50  0000 C CNN
 F 2 "" H 2500 2100 50  0000 C CNN
@@
 Connection ~ 2500 1750
 $Comp
-L VDD #PWR05
+L VDD #PWR12
 U 1 1 574B3528
 P 3400 1550
-F 0 "#PWR05" H 3400 1400 50  0001 C CNN
+F 0 "#PWR12" H 3400 1400 50  0001 C CNN
 F 1 "VDD" H 3420 1724 50  0000 C CNN
 F 2 "" H 3400 1550 50  0000 C CNN
@@
 $EndComp
 $Comp
-L VSS #PWR06
+L VSS #PWR13
 U 1 1 574B3548
 P 3400 2150
-F 0 "#PWR06" H 3400 2000 50  0001 C CNN
+F 0 "#PWR13" H 3400 2000 50  0001 C CNN
 F 1 "VSS" H 3421 2324 50  0000 C CNN
 F 2 "" H 3400 2150 50  0000 C CNN
@@
 	3800 1850 4250 1850
 $Comp
-L GND #PWR07
+L GND #PWR21
 U 1 1 574B35C2
 P 4250 1850
-F 0 "#PWR07" H 4250 1600 50  0001 C CNN
+F 0 "#PWR21" H 4250 1600 50  0001 C CNN
 F 1 "GND" H 4258 1676 50  0000 C CNN
 F 2 "" H 4250 1850 50  0000 C CNN
@@
 $EndComp
 $Comp
-L CONN_01X02 P1
-U 1 1 574B3673
-P 1650 3650
-F 0 "P1" H 1569 3368 50  0000 C CNN
-F 1 "IN" H 1569 3460 50  0000 C CNN
-F 2 "Pin_Headers:Pin_Header_Straight_1x02" H 1650 3650 50  0001 C CNN
-F 3 "" H 1650 3650 50  0000 C CNN
-	1    1650 3650
-	-1   0    0    1
-$EndComp
-$Comp
-L GND #PWR08
+L GND #PWR1
 U 1 1 574B372A
 P 1850 3700
-F 0 "#PWR08" H 1850 3450 50  0001 C CNN
+F 0 "#PWR1" H 1850 3450 50  0001 C CNN
 F 1 "GND" H 1858 3526 50  0000 C CNN
 F 2 "" H 1850 3700 50  0000 C CNN
@@
 $EndComp
 $Comp
-L GND #PWR09
+L GND #PWR6
 U 1 1 574B37E1
 P 2450 3400
-F 0 "#PWR09" H 2450 3150 50  0001 C CNN
+F 0 "#PWR6" H 2450 3150 50  0001 C CNN
 F 1 "GND" H 2458 3226 50  0001 C CNN
 F 2 "" H 2450 3400 50  0000 C CNN
@@
 	2350 3600 2450 3600
 $Comp
-L VSS #PWR010
+L VSS #PWR10
 U 1 1 574B394F
 P 2650 3800
-F 0 "#PWR010" H 2650 3650 50  0001 C CNN
+F 0 "#PWR10" H 2650 3650 50  0001 C CNN
 F 1 "VSS" H 2671 3974 50  0000 C CNN
 F 2 "" H 2650 3800 50  0000 C CNN
@@
 $EndComp
 $Comp
-L VDD #PWR011
+L VDD #PWR9
 U 1 1 574B3986
 P 2650 3200
-F 0 "#PWR011" H 2650 3050 50  0001 C CNN
+F 0 "#PWR9" H 2650 3050 50  0001 C CNN
 F 1 "VDD" H 2670 3374 50  0000 C CNN
 F 2 "" H 2650 3200 50  0000 C CNN
@@
 	3050 3500 3500 3500
 $Comp
-L CONN_01X02 P5
-U 1 1 574B3C13
-P 3850 5400
-F 0 "P5" H 3768 5118 50  0000 C CNN
-F 1 "OUT" H 3768 5210 50  0000 C CNN
-F 2 "Pin_Headers:Pin_Header_Straight_1x02" H 3850 5400 50  0001 C CNN
-F 3 "" H 3850 5400 50  0000 C CNN
-	1    3850 5400
-	1    0    0    1
-$EndComp
-$Comp
-L GND #PWR012
+L GND #PWR16
 U 1 1 574B3CCC
 P 3650 5450
-F 0 "#PWR012" H 3650 5200 50  0001 C CNN
+F 0 "#PWR16" H 3650 5200 50  0001 C CNN
 F 1 "GND" H 3658 5276 50  0000 C CNN
 F 2 "" H 3650 5450 50  0000 C CNN
@@
 $EndComp
 $Comp
-L VDD #PWR013
+L VDD #PWR4
 U 1 1 574B3D47
 P 2400 5050
-F 0 "#PWR013" H 2400 4900 50  0001 C CNN
+F 0 "#PWR4" H 2400 4900 50  0001 C CNN
 F 1 "VDD" H 2420 5224 50  0000 C CNN
 F 2 "" H 2400 5050 50  0000 C CNN
@@
 $EndComp
 $Comp
-L VSS #PWR014
+L VSS #PWR5
 U 1 1 574B3D79
 P 2400 5650
-F 0 "#PWR014" H 2400 5500 50  0001 C CNN
+F 0 "#PWR5" H 2400 5500 50  0001 C CNN
 F 1 "VSS" H 2421 5824 50  0000 C CNN
 F 2 "" H 2400 5650 50  0000 C CNN
@@
 	5350 1800 5550 1800
 $Comp
-L VDD #PWR015
+L VDD #PWR28
 U 1 1 574B52B3
 P 5750 1400
-F 0 "#PWR015" H 5750 1250 50  0001 C CNN
+F 0 "#PWR28" H 5750 1250 50  0001 C CNN
 F 1 "VDD" H 5770 1574 50  0000 C CNN
 F 2 "" H 5750 1400 50  0000 C CNN
@@
 $EndComp
 $Comp
-L VSS #PWR016
+L VSS #PWR29
 U 1 1 574B52F4
 P 5750 2000
-F 0 "#PWR016" H 5750 1850 50  0001 C CNN
+F 0 "#PWR29" H 5750 1850 50  0001 C CNN
 F 1 "VSS" H 5771 2174 50  0000 C CNN
 F 2 "" H 5750 2000 50  0000 C CNN
@@
 	6550 1600 6550 1800
 $Comp
-L VDD #PWR017
+L VDD #PWR30
 U 1 1 574B55CA
 P 5750 2550
-F 0 "#PWR017" H 5750 2400 50  0001 C CNN
+F 0 "#PWR30" H 5750 2400 50  0001 C CNN
 F 1 "VDD" H 5770 2724 50  0000 C CNN
 F 2 "" H 5750 2550 50  0000 C CNN
@@
 $EndComp
 $Comp
-L VSS #PWR018
+L VSS #PWR31
 U 1 1 574B5611
 P 5750 3150
-F 0 "#PWR018" H 5750 3000 50  0001 C CNN
+F 0 "#PWR31" H 5750 3000 50  0001 C CNN
 F 1 "VSS" H 5771 3324 50  0000 C CNN
 F 2 "" H 5750 3150 50  0000 C CNN
@@
 	5350 4150 5550 4150
 $Comp
-L VDD #PWR019
+L VDD #PWR32
 U 1 1 574B5FAA
 P 5750 3750
-F 0 "#PWR019" H 5750 3600 50  0001 C CNN
+F 0 "#PWR32" H 5750 3600 50  0001 C CNN
 F 1 "VDD" H 5770 3924 50  0000 C CNN
 F 2 "" H 5750 3750 50  0000 C CNN
@@
 $EndComp
 $Comp
-L VSS #PWR020
+L VSS #PWR33
 U 1 1 574B5FB0
 P 5750 4350
-F 0 "#PWR020" H 5750 4200 50  0001 C CNN
+F 0 "#PWR33" H 5750 4200 50  0001 C CNN
 F 1 "VSS" H 5771 4524 50  0000 C CNN
 F 2 "" H 5750 4350 50  0000 C CNN
@@
 	6550 3950 6550 4150
 $Comp
-L VDD #PWR021
+L VDD #PWR34
 U 1 1 574B6F19
 P 9450 1650
-F 0 "#PWR021" H 9450 1500 50  0001 C CNN
+F 0 "#PWR34" H 9450 1500 50  0001 C CNN
 F 1 "VDD" H 9470 1824 50  0000 C CNN
 F 2 "" H 9450 1650 50  0000 C CNN
@@
 Connection ~ 9450 1750
 $Comp
-L GND #PWR022
+L GND #PWR35
 U 1 1 574B70C8
 P 9950 2950
-F 0 "#PWR022" H 9950 2700 50  0001 C CNN
+F 0 "#PWR35" H 9950 2700 50  0001 C CNN
 F 1 "GND" H 9958 2776 50  0000 C CNN
 F 2 "" H 9950 2950 50  0000 C CNN
@@
 	10450 1750 10450 2950
 $Comp
-L VSS #PWR023
+L VSS #PWR36
 U 1 1 574B7218
 P 10450 2950
-F 0 "#PWR023" H 10450 2800 50  0001 C CNN
+F 0 "#PWR36" H 10450 2800 50  0001 C CNN
 F 1 "VSS" H 10471 3124 50  0000 C CNN
 F 2 "" H 10450 2950 50  0000 C CNN
@@
 $EndComp
 $Comp
-L VDD #PWR024
+L VDD #PWR24
 U 1 1 574BAC0A
 P 5550 5000
-F 0 "#PWR024" H 5550 4850 50  0001 C CNN
+F 0 "#PWR24" H 5550 4850 50  0001 C CNN
 F 1 "VDD" H 5570 5174 50  0000 C CNN
 F 2 "" H 5550 5000 50  0000 C CNN
@@
 $EndComp
 $Comp
-L VSS #PWR025
+L VSS #PWR25
 U 1 1 574BAC10
 P 5550 5600
-F 0 "#PWR025" H 5550 5450 50  0001 C CNN
+F 0 "#PWR25" H 5550 5450 50  0001 C CNN
 F 1 "VSS" H 5571 5774 50  0000 C CNN
 F 2 "" H 5550 5600 50  0000 C CNN
@@
 	5150 6600 5350 6600
 $Comp
-L VDD #PWR026
+L VDD #PWR26
 U 1 1 574BAC29
 P 5550 6200
-F 0 "#PWR026" H 5550 6050 50  0001 C CNN
+F 0 "#PWR26" H 5550 6050 50  0001 C CNN
 F 1 "VDD" H 5570 6374 50  0000 C CNN
 F 2 "" H 5550 6200 50  0000 C CNN
@@
 $EndComp
 $Comp
-L VSS #PWR027
+L VSS #PWR27
 U 1 1 574BAC2F
 P 5550 6800
-F 0 "#PWR027" H 5550 6650 50  0001 C CNN
+F 0 "#PWR27" H 5550 6650 50  0001 C CNN
 F 1 "VSS" H 5571 6974 50  0000 C CNN
 F 2 "" H 5550 6800 50  0000 C CNN
@@
 $EndComp
 $Comp
-L VDD #PWR028
+L VDD #PWR14
 U 1 1 574BC4E6
 P 3600 850
-F 0 "#PWR028" H 3600 700 50  0001 C CNN
+F 0 "#PWR14" H 3600 700 50  0001 C CNN
 F 1 "VDD" H 3620 1024 50  0000 C CNN
 F 2 "" H 3600 850 50  0000 C CNN
@@
 $EndComp
 $Comp
-L VDD #PWR029
+L VDD #PWR17
 U 1 1 574BC587
 P 3900 850
-F 0 "#PWR029" H 3900 700 50  0001 C CNN
+F 0 "#PWR17" H 3900 700 50  0001 C CNN
 F 1 "VDD" H 3920 1024 50  0000 C CNN
 F 2 "" H 3900 850 50  0000 C CNN
@@
 $EndComp
 $Comp
-L VDD #PWR030
+L VDD #PWR19
 U 1 1 574BC628
 P 4200 850
-F 0 "#PWR030" H 4200 700 50  0001 C CNN
+F 0 "#PWR19" H 4200 700 50  0001 C CNN
 F 1 "VDD" H 4220 1024 50  0000 C CNN
 F 2 "" H 4200 850 50  0000 C CNN
@@
 $EndComp
 $Comp
-L VDD #PWR031
+L VDD #PWR22
 U 1 1 574BC6C9
 P 4500 850
-F 0 "#PWR031" H 4500 700 50  0001 C CNN
+F 0 "#PWR22" H 4500 700 50  0001 C CNN
 F 1 "VDD" H 4520 1024 50  0000 C CNN
 F 2 "" H 4500 850 50  0000 C CNN
@@
 $EndComp
 $Comp
-L VSS #PWR032
+L VSS #PWR15
 U 1 1 574BC76A
 P 3600 1150
-F 0 "#PWR032" H 3600 1000 50  0001 C CNN
+F 0 "#PWR15" H 3600 1000 50  0001 C CNN
 F 1 "VSS" H 3621 1324 50  0000 C CNN
 F 2 "" H 3600 1150 50  0000 C CNN
@@
 $EndComp
 $Comp
-L VSS #PWR033
+L VSS #PWR18
 U 1 1 574BC869
 P 3900 1150
-F 0 "#PWR033" H 3900 1000 50  0001 C CNN
+F 0 "#PWR18" H 3900 1000 50  0001 C CNN
 F 1 "VSS" H 3921 1324 50  0000 C CNN
 F 2 "" H 3900 1150 50  0000 C CNN
@@
 $EndComp
 $Comp
-L VSS #PWR034
+L VSS #PWR20
 U 1 1 574BC968
 P 4200 1150
-F 0 "#PWR034" H 4200 1000 50  0001 C CNN
+F 0 "#PWR20" H 4200 1000 50  0001 C CNN
 F 1 "VSS" H 4221 1324 50  0000 C CNN
 F 2 "" H 4200 1150 50  0000 C CNN
@@
 $EndComp
 $Comp
-L VSS #PWR035
+L VSS #PWR23
 U 1 1 574BCA67
 P 4500 1150
-F 0 "#PWR035" H 4500 1000 50  0001 C CNN
+F 0 "#PWR23" H 4500 1000 50  0001 C CNN
 F 1 "VSS" H 4521 1324 50  0000 C CNN
 F 2 "" H 4500 1150 50  0000 C CNN
@@
 Connection ~ 2850 1750
 $Comp
-L VSS #PWR036
+L VSS #PWR11
 U 1 1 574BACA1
 P 2850 2100
-F 0 "#PWR036" H 2850 1950 50  0001 C CNN
+F 0 "#PWR11" H 2850 1950 50  0001 C CNN
 F 1 "VSS" H 2871 2274 50  0000 C CNN
 F 2 "" H 2850 2100 50  0000 C CNN
@@
 	-1   0    0    1
 $EndComp
+$Comp
+L CONN_01X03 P1
+U 1 1 574C48D1
+P 1650 3600
+F 0 "P1" H 1569 3268 50  0000 C CNN
+F 1 "IN" H 1569 3360 50  0000 C CNN
+F 2 "Pin_Headers:Pin_Header_Straight_1x03" H 1650 3600 50  0001 C CNN
+F 3 "" H 1650 3600 50  0000 C CNN
+	1    1650 3600
+	-1   0    0    1
+$EndComp
+Wire Wire Line
+	1850 3500 1900 3500
+Wire Wire Line
+	1900 3500 1900 3600
+Connection ~ 1900 3600
+$Comp
+L CONN_01X03 P5
+U 1 1 574C5765
+P 3850 5350
+F 0 "P5" H 3927 5388 50  0000 L CNN
+F 1 "OUT" H 3927 5296 50  0000 L CNN
+F 2 "Pin_Headers:Pin_Header_Straight_1x03" H 3850 5350 50  0001 C CNN
+F 3 "" H 3850 5350 50  0000 C CNN
+	1    3850 5350
+	1    0    0    1
+$EndComp
+Wire Wire Line
+	3650 5250 3550 5250
+Wire Wire Line
+	3550 5250 3550 5350
+Connection ~ 3550 5350
 $EndSCHEMATC

Commit message: Final tweaks
Parts:
- added C6: 100n, agg:0603, symbol C
- added D1: LED, Pin_Headers:Pin_Header_Straight_1x02, symbol LED
- added R5: R, agg:0603, symbol R
Connections:
- net GND: now also C6.1
- net VDD: now also R5.1
- net VSS: now also C6.2, D1.1 (K)
- new net: D1.2 (A), R5.2
Other:
- moved on the sheet: P3

Commit message: Added farnell parts, removed unfitted LED
Parts:
- removed D1: LED, Pin_Headers:Pin_Header_Straight_1x02, symbol LED
- removed R5: R, agg:0603, symbol R
- C1, C2, C3, C4, C5, C6: Farnell (none) -> 2524817
- R1, R4: Farnell (none) -> 9330410
- R2, R3: Farnell (none) -> 2309107
- U1, U2, U3, U4: value LM358N -> LM358; Farnell (none) -> 2342291
