File: dsp/dsp.kicad_pcb (KiCad board)
At the start: 2 copper layers, 50 x 50 mm, 43 parts, among them IC1 STM32F405RxTx, P1 IN, P2 BATT_IN, P3 ENCODER, P4 SWD_TC, P5 OUT, P7 CONN_01X07, SW1 SPST, U1 NCP1117, U2 LM358N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

Commit message: Final tweaks
Parts:
- added C17: 100n, agg:0603, F.Cu at (154.9, 67.1)
- added C18: 100n, agg:0603, F.Cu at (163.6, 69.6)
- added D2: LED, Pin_Headers:Pin_Header_Straight_1x02, F.Cu at (195.1, 63.2)
- added R8: R, agg:0603, F.Cu at (192.5, 62.2)
- R2: value 100k -> 82k5
- R3: value 100k -> 18k7
Routing:
- net +3V3: track 186.2 -> 193.4 mm
- net VSS: track 65.5 -> 68.4 mm
- net Net-(D2-Pad2): track 0.00 -> 2.84 mm
- net VDD: track 36.8 -> 39.2 mm
- net GND: track 5.46 -> 6.69 mm, vias 2 -> 3
- net Net-(C3-Pad1): track 12.7 -> 13.7 mm
- net /nRST: track 24.8 -> 25.6 mm
Other:
- board text added: "DAVID TURNER"
- board text added: "LED"
- board text removed: "David Turner"
